File: elec/layout/default/project.kicad_pcb (KiCad board)
At the start: 2 copper layers, 40 x 40 mm, 0 parts

Commit message: Configure project
Other:
- board text added: "{{GITHASH}}"
- board text removed: "{{"
Changed lines of the file:
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@@
 		(layer "Edge.Cuts")
 	)
-	(gr_text "{{"{{GITHASH}}"}}"
+	(gr_text "{{GITHASH}}"
 		(at 140.240427 116.111573 0)
 		(layer "F.SilkS")
