File: kicad/mcu_core.kicad_sch (KiCad schematic)
At the start: 39 parts, among them J10 SWD, SW1 BOOTSEL, SW2 RESET, U1 RP2350B, U2 W25Q128JVS, U3 DNP second memory, Y1 ABM8-272-T3

Commit message: Pick JLCPCB parts for the whole BOM and add BOM/CPL generation
Adds bom/parts.csv (LCSC numbers and MPNs), scripts to apply it to the schematic and
board and to generate the JLCPCB BOM, CPL and a live stock report. Swaps the
BOOTSEL/RESET switch to a basic 5.1 mm part with a matching footprint, and replaces
out-of-stock parts (SS54, WS2812B, 10u caps, SWD header).

Co-Authored-By: Claude Sonnet 5.5 <noreply@anthropic.com>
Parts:
- C1, C2, C5, C6: LCSC (none) -> C23733; MPN (none) -> CL05A475MP5NRNC
- C10, C11, C12, C13, C14, C15, C19, C20, C3, C4, C7, C8, C9: LCSC (none) -> C307331; MPN (none) -> CL05B104KB54PNC
- C16: LCSC (none) -> C15850; MPN (none) -> CL21A106KAYNNNE
- C17, C18: LCSC (none) -> C106997; MPN (none) -> CC0402JRNPO9BN150
- J10: LCSC (none) -> C239521; MPN SM03B-SRSS-TB -> A1002WR-S-3P
- L1: LCSC (none) -> C42411119
- R1: LCSC (none) -> C25105; MPN (none) -> 0402WGF330JTCE
- R10, R11: LCSC (none) -> C25100; MPN (none) -> 0402WGF270JTCE
- R2, R8, R9: LCSC (none) -> C11702; MPN (none) -> 0402WGF1001TCE
- R3, R5, R6: LCSC (none) -> C17168; MPN (none) -> 0402WGF0000TCE
- R4, R7: LCSC (none) -> C25744; MPN (none) -> 0402WGF1002TCE
- SW1, SW2: footprint Button_Switch_SMD:SW_Push_1P1T_NO_Vertical_Wuerth_434133025816 -> picomondo:SW_SMD_TS-1187A_5.1x5.1; LCSC (none) -> C318884; MPN B3FS-4005P -> TS-1187A-B-A-B
- U1: LCSC (none) -> C42415655
- U2: LCSC (none) -> C97521; MPN W25Q128JVS -> W25Q128JVSIQ
- Y1: LCSC (none) -> C20625731

Commit message: Rework board layout, swap SWD header to through-hole, add Qwiic port
- SWD (J10) is now a 1x3 2.54 mm through-hole pin header footprint
  (SWCLK, GND, SWDIO) instead of the JST SH connector; removed from the
  JLCPCB BOM.
- Add J20 Qwiic connector (XY-SM04B-SRSS-TB) on the I2C bus: GND, +3V3,
  GPIO20 (SDA), GPIO21 (SCL), mounting tabs to GND.
- Placement/routing progress and the helper scripts used for it.

DRC still reports open items (unrouted RUN/GPIO24/GPIO29/QSPI_SD0 nets,
R108/GPIO23 and NT1/GPIO20 shorts, J12 edge clearance, silkscreen
overlaps); to be fixed in follow-up commits.

Co-Authored-By: Claude Sonnet 5.5 <noreply@anthropic.com>
Parts:
- J10: footprint Connector_JST:JST_SH_SM03B-SRSS-TB_1x03-1MP_P1.00mm_Horizontal -> Connector_PinHeader_2.54mm:PinHeader_1x03_P2.54mm_Horizontal; MPN A1002WR-S-3P -> (none); now not fitted; now left out of the parts list
- U3: now fitted
