File: kicad/power_buck.kicad_sch (KiCad schematic)
At the start: 33 parts, among them Q1 CSD18543Q3A, Q2 CSD18543Q3A, U4 TPS55288

Commit message: Pick JLCPCB parts for the whole BOM and add BOM/CPL generation
Adds bom/parts.csv (LCSC numbers and MPNs), scripts to apply it to the schematic and
board and to generate the JLCPCB BOM, CPL and a live stock report. Swaps the
BOOTSEL/RESET switch to a basic 5.1 mm part with a matching footprint, and replaces
out-of-stock parts (SS54, WS2812B, 10u caps, SWD header).

Co-Authored-By: Claude Sonnet 5.5 <noreply@anthropic.com>
Parts:
- C25, C27, C28, C33: LCSC (none) -> C307331; MPN (none) -> CL05B104KB54PNC
- C36: LCSC (none) -> C15850; MPN (none) -> CL21A106KAYNNNE
- C37: LCSC (none) -> C15195; MPN (none) -> CL05B103KB5NNNC
- C38: LCSC (none) -> C26404; MPN (none) -> CL05B332KB5NNNC
- R13: LCSC (none) -> C25897; MPN (none) -> 0402WGF4992TCE
- R14: LCSC (none) -> C122548; MPN (none) -> 0402WGF3322TCE
- R15: LCSC (none) -> C25741; MPN (none) -> 0402WGF1003TCE
- R16: LCSC (none) -> C17168; MPN (none) -> 0402WGF0000TCE
- R17: LCSC (none) -> C25918; MPN (none) -> 0402WGF7501TCE
- R18: LCSC (none) -> C25767; MPN (none) -> 0402WGF2203TCE
- R19: LCSC (none) -> C25922; MPN (none) -> 0402WGF8872TCE
- R20: LCSC (none) -> C25744; MPN (none) -> 0402WGF1002TCE
Changed lines of the file:
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@@
     (stroke (width 0) (type default))
   )
-  (wire (pts (xy 254.0 212.09) (xy 254.0 207.01))
+  (wire (pts (xy 254 212.09) (xy 254 207.01))
     (stroke (width 0) (type default))
   )
-  (wire (pts (xy 254.0 219.71) (xy 264.16 219.71))
+  (wire (pts (xy 254 219.71) (xy 264.16 219.71))
     (stroke (width 0) (type default))
   )
@@
   )
   (text "POWER STAGE: keep V_INPUT -> Q1 -> Q2 -> GND -> input caps loop tiny; SW1/SW2 traces short and wide,\ntop layer, no vias. Inductor: 4.7 uH, saturation current 12 A or more, DCR 12 mohm or less\n(Coilcraft XAL1010-472 or equivalent). 0.1 uF bootstrap caps right at BOOT/SW pins."
-    (at 114.3 160.0 0)
+    (at 114.3 160 0)
     (effects (font (size 1.8 1.8)) (justify left))
   )
@@
     )
   )
-  (global_label "V_INPUT" (shape bidirectional) (at 254.0 207.01 90)
-    (effects (font (size 1.27 1.27)))
-    (property "Intersheetrefs" "${INTERSHEET_REFS}" (id 0) (at 254.0 207.01 0)
+  (global_label "V_INPUT" (shape bidirectional) (at 254 207.01 90)
+    (effects (font (size 1.27 1.27)))
+    (property "Intersheetrefs" "${INTERSHEET_REFS}" (id 0) (at 254 207.01 0)
       (effects (font (size 1.27 1.27)) hide)
     )
@@
       (effects (font (size 1.27 1.27)) hide)
     )
+    (property "LCSC" "C307331" (id 4) (at 89.535 60.96 0)
+      (effects (font (size 1.27 1.27)) hide)
+    )
+    (property "MPN" "CL05B104KB54PNC" (id 5) (at 89.535 60.96 0)
+      (effects (font (size 1.27 1.27)) hide)
+    )
     (pin "1")
     (pin "2")
@@
     )
   )
-  (symbol (lib_id "lcsc:CSD18543Q3A") (at 152.4 127.0 0) (unit 1)
+  (symbol (lib_id "lcsc:CSD18543Q3A") (at 152.4 127 0) (unit 1)
     (in_bom yes) (on_board yes) (dnp no)
     (property "Reference" "Q2" (id 0) (at 152.4 115.57 0)
@@
       (effects (font (size 1.27 1.27)) hide)
     )
-    (property "Datasheet" "" (id 3) (at 152.4 127.0 0)
-      (effects (font (size 1.27 1.27)) hide)
-    )
-    (property "MPN" "CSD18543Q3A" (id 4) (at 152.4 127.0 0)
-      (effects (font (size 1.27 1.27)) hide)
-    )
-    (property "LCSC" "C840100" (id 5) (at 152.4 127.0 0)
+    (property "Datasheet" "" (id 3) (at 152.4 127 0)
+      (effects (font (size 1.27 1.27)) hide)
+    )
+    (property "MPN" "CSD18543Q3A" (id 4) (at 152.4 127 0)
+      (effects (font (size 1.27 1.27)) hide)
+    )
+    (property "LCSC" "C840100" (id 5) (at 152.4 127 0)
       (effects (font (size 1.27 1.27)) hide)
     )
@@
       (effects (font (size 1.27 1.27)) hide)
     )
+    (property "LCSC" "C307331" (id 4) (at 191.135 60.96 0)
+      (effects (font (size 1.27 1.27)) hide)
+    )
+    (property "MPN" "CL05B104KB54PNC" (id 5) (at 191.135 60.96 0)
+      (effects (font (size 1.27 1.27)) hide)
+    )
     (pin "1")
     (pin "2")
@@
       (effects (font (size 1.27 1.27)) hide)
     )
+    (property "LCSC" "C307331" (id 4) (at 216.535 60.96 0)
+      (effects (font (size 1.27 1.27)) hide)
+    )
+    (property "MPN" "CL05B104KB54PNC" (id 5) (at 216.535 60.96 0)
+      (effects (font (size 1.27 1.27)) hide)
+    )
     (pin "1")
     (pin "2")
@@
       (effects (font (size 1.27 1.27)) hide)
     )
+    (property "LCSC" "C307331" (id 4) (at 451.485 99.06 0)
+      (effects (font (size 1.27 1.27)) hide)
+    )
+    (property "MPN" "CL05B104KB54PNC" (id 5) (at 451.485 99.06 0)
+      (effects (font (size 1.27 1.27)) hide)
+    )
     (pin "1")
     (pin "2")
@@
       (effects (font (size 1.27 1.27)) hide)
     )
+    (property "LCSC" "C15850" (id 4) (at 64.135 213.36 0)
+      (effects (font (size 1.27 1.27)) hide)
+    )
+    (property "MPN" "CL21A106KAYNNNE" (id 5) (at 64.135 213.36 0)
+      (effects (font (size 1.27 1.27)) hide)
+    )
     (pin "1")
     (pin "2")
@@
       (effects (font (size 1.27 1.27)) hide)
     )
+    (property "LCSC" "C25897" (id 4) (at 90.932 215.9 0)
+      (effects (font (size 1.27 1.27)) hide)
+    )
+    (property "MPN" "0402WGF4992TCE" (id 5) (at 90.932 215.9 0)
+      (effects (font (size 1.27 1.27)) hide)
+    )
     (pin "1")
     (pin "2")
@@
       (effects (font (size 1.27 1.27)) hide)
     )
+    (property "LCSC" "C15195" (id 4) (at 114.935 213.36 0)
+      (effects (font (size 1.27 1.27)) hide)
+    )
+    (property "MPN" "CL05B103KB5NNNC" (id 5) (at 114.935 213.36 0)
+      (effects (font (size 1.27 1.27)) hide)
+    )
     (pin "1")
     (pin "2")
@@
       (effects (font (size 1.27 1.27)) hide)
     )
+    (property "LCSC" "C122548" (id 4) (at 141.732 215.9 0)
+      (effects (font (size 1.27 1.27)) hide)
+    )
+    (property "MPN" "0402WGF3322TCE" (id 5) (at 141.732 215.9 0)
+      (effects (font (size 1.27 1.27)) hide)
+    )
     (pin "1")
     (pin "2")
@@
       (effects (font (size 1.27 1.27)) hide)
     )
+    (property "LCSC" "C25741" (id 4) (at 167.132 215.9 0)
+      (effects (font (size 1.27 1.27)) hide)
+    )
+    (property "MPN" "0402WGF1003TCE" (id 5) (at 167.132 215.9 0)
+      (effects (font (size 1.27 1.27)) hide)
+    )
     (pin "1")
     (pin "2")
@@
       (effects (font (size 1.27 1.27)) hide)
     )
+    (property "LCSC" "C17168" (id 5) (at 192.532 215.9 0)
+      (effects (font (size 1.27 1.27)) hide)
+    )
+    (property "MPN" "0402WGF0000TCE" (id 6) (at 192.532 215.9 0)
+      (effects (font (size 1.27 1.27)) hide)
+    )
     (pin "1")
     (pin "2")
@@
       (effects (font (size 1.27 1.27)) hide)
     )
+    (property "LCSC" "C25918" (id 4) (at 217.932 215.9 0)
+      (effects (font (size 1.27 1.27)) hide)
+    )
+    (property "MPN" "0402WGF7501TCE" (id 5) (at 217.932 215.9 0)
+      (effects (font (size 1.27 1.27)) hide)
+    )
     (pin "1")
     (pin "2")
@@
     )
     (property "Datasheet" "" (id 3) (at 215.9 223.52 0)
+      (effects (font (size 1.27 1.27)) hide)
+    )
+    (property "LCSC" "C26404" (id 4) (at 216.535 220.98 0)
+      (effects (font (size 1.27 1.27)) hide)
+    )
+    (property "MPN" "CL05B332KB5NNNC" (id 5) (at 216.535 220.98 0)
       (effects (font (size 1.27 1.27)) hide)
     )
@@
     )
   )
-  (symbol (lib_id "Device:R") (at 254.0 215.9 0) (unit 1)
+  (symbol (lib_id "Device:R") (at 254 215.9 0) (unit 1)
     (in_bom yes) (on_board yes) (dnp no)
     (property "Reference" "R18" (id 0) (at 256.032 215.9 90)
       (effects (font (size 1.27 1.27)))
     )
-    (property "Value" "220k 1%" (id 1) (at 254.0 215.9 90)
+    (property "Value" "220k 1%" (id 1) (at 254 215.9 90)
       (effects (font (size 1.27 1.27)))
     )
@@
       (effects (font (size 1.27 1.27)) hide)
     )
-    (property "Datasheet" "" (id 3) (at 254.0 215.9 0)
+    (property "Datasheet" "" (id 3) (at 254 215.9 0)
+      (effects (font (size 1.27 1.27)) hide)
+    )
+    (property "LCSC" "C25767" (id 4) (at 256.032 215.9 0)
+      (effects (font (size 1.27 1.27)) hide)
+    )
+    (property "MPN" "0402WGF2203TCE" (id 5) (at 256.032 215.9 0)
       (effects (font (size 1.27 1.27)) hide)
     )
@@
     )
   )
-  (symbol (lib_id "Device:R") (at 254.0 223.52 0) (unit 1)
+  (symbol (lib_id "Device:R") (at 254 223.52 0) (unit 1)
     (in_bom yes) (on_board yes) (dnp no)
     (property "Reference" "R19" (id 0) (at 256.032 223.52 90)
       (effects (font (size 1.27 1.27)))
     )
-    (property "Value" "88.7k 1%" (id 1) (at 254.0 223.52 90)
+    (property "Value" "88.7k 1%" (id 1) (at 254 223.52 90)
       (effects (font (size 1.27 1.27)))
     )
@@
       (effects (font (size 1.27 1.27)) hide)
     )
-    (property "Datasheet" "" (id 3) (at 254.0 223.52 0)
+    (property "Datasheet" "" (id 3) (at 254 223.52 0)
+      (effects (font (size 1.27 1.27)) hide)
+    )
+    (property "LCSC" "C25922" (id 4) (at 256.032 223.52 0)
+      (effects (font (size 1.27 1.27)) hide)
+    )
+    (property "MPN" "0402WGF8872TCE" (id 5) (at 256.032 223.52 0)
       (effects (font (size 1.27 1.27)) hide)
     )
@@
     )
   )
-  (symbol (lib_id "power:GNDA") (at 254.0 227.33 0) (unit 1)
-    (in_bom no) (on_board no) (dnp no)
-    (property "Reference" "#PWR3030" (id 0) (at 254.0 233.68 0)
-      (effects (font (size 1.27 1.27)) hide)
-    )
-    (property "Value" "AGND" (id 1) (at 254.0 231.14 0)
-      (effects (font (size 1.27 1.27)))
-    )
-    (property "Footprint" "" (id 2) (at 254.0 227.33 0)
-      (effects (font (size 1.27 1.27)) hide)
-    )
-    (property "Datasheet" "" (id 3) (at 254.0 227.33 0)
+  (symbol (lib_id "power:GNDA") (at 254 227.33 0) (unit 1)
+    (in_bom no) (on_board no) (dnp no)
+    (property "Reference" "#PWR3030" (id 0) (at 254 233.68 0)
+      (effects (font (size 1.27 1.27)) hide)
+    )
+    (property "Value" "AGND" (id 1) (at 254 231.14 0)
+      (effects (font (size 1.27 1.27)))
+    )
+    (property "Footprint" "" (id 2) (at 254 227.33 0)
+      (effects (font (size 1.27 1.27)) hide)
+    )
+    (property "Datasheet" "" (id 3) (at 254 227.33 0)
       (effects (font (size 1.27 1.27)) hide)
     )
@@
       (effects (font (size 1.27 1.27)) hide)
     )
+    (property "LCSC" "C25744" (id 4) (at 281.432 215.9 0)
+      (effects (font (size 1.27 1.27)) hide)
+    )
+    (property "MPN" "0402WGF1002TCE" (id 5) (at 281.432 215.9 0)
+      (effects (font (size 1.27 1.27)) hide)
+    )

Commit message: Rework board layout, swap SWD header to through-hole, add Qwiic port
- SWD (J10) is now a 1x3 2.54 mm through-hole pin header footprint
  (SWCLK, GND, SWDIO) instead of the JST SH connector; removed from the
  JLCPCB BOM.
- Add J20 Qwiic connector (XY-SM04B-SRSS-TB) on the I2C bus: GND, +3V3,
  GPIO20 (SDA), GPIO21 (SCL), mounting tabs to GND.
- Placement/routing progress and the helper scripts used for it.

DRC still reports open items (unrouted RUN/GPIO24/GPIO29/QSPI_SD0 nets,
R108/GPIO23 and NT1/GPIO20 shorts, J12 edge clearance, silkscreen
overlaps); to be fixed in follow-up commits.

Co-Authored-By: Claude Sonnet 5.5 <noreply@anthropic.com>
Parts:
- C26: now fitted
