File: kicad/power_ldo.kicad_sch (KiCad schematic)
At the start: 6 parts, among them U5 AP2112K-3.3, U6 AP2112K-3.3

Commit message: Pick JLCPCB parts for the whole BOM and add BOM/CPL generation
Adds bom/parts.csv (LCSC numbers and MPNs), scripts to apply it to the schematic and
board and to generate the JLCPCB BOM, CPL and a live stock report. Swaps the
BOOTSEL/RESET switch to a basic 5.1 mm part with a matching footprint, and replaces
out-of-stock parts (SS54, WS2812B, 10u caps, SWD header).

Co-Authored-By: Claude Sonnet 5.5 <noreply@anthropic.com>
Parts:
- C40, C41, C42, C43: LCSC C91158 -> C15850; MPN (none) -> CL21A106KAYNNNE
Changed lines of the file:
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@@
   )
   (text "+3V3: MCU, flash, microSD, indicators, connector 3.3 V pins.\nTHERMAL LIMIT: 1.7 V x load current is dissipated here (SOT-23-5, 184 C/W in the datasheet).\nAt 40 C ambient that allows about 350 mA unless the pad is tied to a large copper area.\nBudget: MCU about 100 mA, flash 20 mA, microSD up to 100 mA, connector loads on top."
-    (at 50.800000000000004 127.0 0)
+    (at 50.800000000000004 127 0)
     (effects (font (size 1.8 1.8)) (justify left))
   )
@@
       (effects (font (size 1.27 1.27)) hide)
     )
-    (property "LCSC" "C91158" (id 4) (at 63.50000000000001 83.82000000000001 0)
+    (property "LCSC" "C15850" (id 4) (at 63.50000000000001 83.82000000000001 0)
+      (effects (font (size 1.27 1.27)) hide)
+    )
+    (property "MPN" "CL21A106KAYNNNE" (id 5) (at 64.135 81.28 0)
       (effects (font (size 1.27 1.27)) hide)
     )
@@
       (effects (font (size 1.27 1.27)) hide)
     )
-    (property "LCSC" "C91158" (id 4) (at 114.30000000000001 83.82000000000001 0)
+    (property "LCSC" "C15850" (id 4) (at 114.30000000000001 83.82000000000001 0)
+      (effects (font (size 1.27 1.27)) hide)
+    )
+    (property "MPN" "CL21A106KAYNNNE" (id 5) (at 114.935 81.28 0)
       (effects (font (size 1.27 1.27)) hide)
     )
@@
       (effects (font (size 1.27 1.27)) hide)
     )
-    (property "LCSC" "C91158" (id 4) (at 63.50000000000001 160.02 0)
+    (property "LCSC" "C15850" (id 4) (at 63.50000000000001 160.02 0)
+      (effects (font (size 1.27 1.27)) hide)
+    )
+    (property "MPN" "CL21A106KAYNNNE" (id 5) (at 64.135 157.48 0)
       (effects (font (size 1.27 1.27)) hide)
     )
@@
       (effects (font (size 1.27 1.27)) hide)
     )
-    (property "LCSC" "C91158" (id 4) (at 114.30000000000001 160.02 0)
-      (effects (font (size 1.27 1.27)) hide)
-    )
+    (property "LCSC" "C15850" (id 4) (at 114.30000000000001 160.02 0)
+      (effects (font (size 1.27 1.27)) hide)
+    )
+    (property "MPN" "CL21A106KAYNNNE" (id 5) (at 114.935 157.48 0)
+      (effects (font (size 1.27 1.27)) hide)
+    )
